File: charger2.kicad_pcb (KiCad board)
At the start: 2 copper layers, 45.7 x 27.9 mm, 15 parts, among them IC1 BQ25606RGER, J1 Screw_Terminal_01x05, J2 Screw_Terminal_01x05, J3 Conn_01x01_Male

Commit message: autorouted
Parts:
- C1: footprint 1uF cap:C1206 -> Library:C1206
- C2: footprint cap 4.7uf:C1210 -> Library:C1210
- C3: footprint 47nF:C1005_Commercial -> Library:C1005_Commercial
- C4, C5: footprint 10uF MLCC:CAPC2012X94N -> Library:CAPC2012X94N
- IC1: footprint BQ25606:QFN50P400X400X100-25N-D -> Library:QFN50P400X400X100-25N-D
- J1, J2: footprint TerminalBlock_MetzConnect:TerminalBlock_MetzConnect_Type059_RT06305HBWC_1x05_P3.50mm_Horizontal -> Library:TerminalBlock_MetzConnect_Type059_RT06305HBWC_1x05_P3.50mm_Horizontal
- J3: footprint Connector_PinHeader_1.00mm:PinHeader_1x01_P1.00mm_Vertical -> Library:PinHeader_1x01_P1.00mm_Vertical
- L1: footprint 1uH indc:IHHP0805ZHER1R0M01 -> Library:IHHP0805ZHER1R0M01
- R1, R2: footprint 2.2k rst:RESC2012X65N -> Library:RESC2012X65N
- R3: footprint rst 330:H2C_H2R -> Library:H2C_H2R
- R4: footprint 10k rst:ERA8KEB1004V -> Library:ERA8KEB1004V
- R5: footprint rst 430:ERJH3 -> Library:ERJH3
- moved J2 36.9 mm to (165.1, 101.6), turned to -90 degrees
- moved R1 24.0 mm to (139.7, 108.7)
- moved R4 24.0 mm to (154.9, 116.8)
- moved C3 18.7 mm to (147.3, 101.6)
- moved C2 17.6 mm to (143.5, 104.1), turned to 90 degrees
- moved C4 14.9 mm to (150.7, 101.0), turned to 180 degrees
- moved C1 13.7 mm to (138.9, 104.1), turned to 90 degrees
- moved J3 12.7 mm to (149.9, 116.8)
- moved J1 12.0 mm to (130.9, 116.9), turned to 90 degrees
- moved R2 10.2 mm to (145.7, 111.4)
- moved IC1 8.07 mm to (149.9, 106.7)
- moved C5 7.86 mm to (154.9, 106.7), turned to 90 degrees
- moved R3 7.40 mm to (148.8, 111.8), turned to -90 degrees
- moved R5 5.20 mm to (152.4, 111.8)
- moved L1 5.16 mm to (154.0, 102.2), turned to -90 degrees
Routing:
- net Earth: track 0.00 -> 112.9 mm
- net Net-(IC1-Pad15): track 0.00 -> 25.2 mm
- net Net-(C2-Pad2): track 0.00 -> 21.4 mm
- net Net-(C1-Pad2): track 0.00 -> 20.8 mm
- net Net-(IC1-Pad11): track 0.00 -> 17.8 mm
- net Net-(R2-Pad2): track 0.00 -> 17.0 mm
- net Net-(IC1-Pad5): track 0.00 -> 16.5 mm
- net Net-(C5-Pad1): track 0.00 -> 16.4 mm
- net Net-(C3-Pad2): track 0.00 -> 14.2 mm
- net Net-(IC1-Pad9): track 0.00 -> 11.8 mm
- net Net-(C4-Pad2): track 0.00 -> 11.3 mm, vias 0 -> 2
- net Net-(R1-Pad2): track 0.00 -> 10.6 mm
- net Net-(IC1-Pad7): track 0.00 -> 5.40 mm
- net Net-(C3-Pad1): track 0.00 -> 5.33 mm
- net Net-(IC1-Pad10): track 0.00 -> 4.11 mm
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
Commit message: patch
Routing:
- net Net-(C2-Pad2): track 21.4 -> 22.4 mm
- net Earth: track 112.9 -> 113.4 mm
Changed lines of the file:
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@@
   (gr_line (start 170.18 127) (end 124.46 127) (layer "Edge.Cuts") (width 0.1))
   (segment (start 153.7751 111.76) (end 154.8275 112.8124) (width 0.25) (layer "F.Cu") (net 1))
+  (segment (start 129.4119 112.7693) (end 130.5162 111.665) (width 0.25) (layer "F.Cu") (net 1))
   (segment (start 157.6151 116.84) (end 157.909 117.1339) (width 0.25) (layer "F.Cu") (net 1))
   (segment (start 151.6788 105.43) (end 151.4975 105.43) (width 0.25) (layer "F.Cu") (net 1))
@@
   (segment (start 156.665 116.84) (end 157.6151 116.84) (width 0.25) (layer "F.Cu") (net 1))
   (segment (start 166.5992 116.2579) (end 166.5992 107.3488) (width 0.25) (layer "F.Cu") (net 1))
-  (segment (start 139.3607 111.665) (end 130.5162 111.665) (width 0.25) (layer "F.Cu") (net 1))
+  (segment (start 130.887 116.1774) (end 130.887 115.4399) (width 0.25) (layer "F.Cu") (net 1))
   (segment (start 151.6788 105.43) (end 151.6788 102.2339) (width 0.25) (layer "F.Cu") (net 1))
-  (segment (start 144.0078 107.0179) (end 139.3607 111.665) (width 0.25) (layer "F.Cu") (net 1))
   (segment (start 151.7694 105.43) (end 151.86 105.43) (width 0.25) (layer "F.Cu") (net 1))
-  (segment (start 129.4119 112.7693) (end 129.4119 114.0571) (width 0.25) (layer "F.Cu") (net 1))
+  (segment (start 130.7947 115.4399) (end 129.4119 114.0571) (width 0.25) (layer "F.Cu") (net 1))
   (segment (start 154.8275 117.1026) (end 154.0149 117.9152) (width 0.25) (layer "F.Cu") (net 1))
   (segment (start 154.0149 117.9152) (end 149.584 117.9152) (width 0.25) (layer "F.Cu") (net 1))
   (segment (start 156.4275 116.84) (end 156.665 116.84) (width 0.25) (layer "F.Cu") (net 1))
-  (segment (start 129.4119 114.0571) (end 130.7947 115.4399) (width 0.25) (layer "F.Cu") (net 1))
   (segment (start 165.7232 117.1339) (end 166.5992 116.2579) (width 0.25) (layer "F.Cu") (net 1))
+  (segment (start 139.515 111.665) (end 143.25 107.93) (width 0.25) (layer "F.Cu") (net 1))
   (segment (start 156.0205 105.8496) (end 156.0001 105.87) (width 0.25) (layer "F.Cu") (net 1))
-  (segment (start 130.5162 111.665) (end 129.4119 112.7693) (width 0.25) (layer "F.Cu") (net 1))
   (segment (start 138.9 105.64) (end 143.53 105.64) (width 0.25) (layer "F.Cu") (net 1))
   (segment (start 151.3411 105.43) (end 151.1349 105.6362) (width 0.25) (layer "F.Cu") (net 1))
+  (segment (start 143.25 107.93) (end 144.9199 107.93) (width 0.25) (layer "F.Cu") (net 1))
   (segment (start 154.8275 112.8124) (end 154.8275 116.84) (width 0.25) (layer "F.Cu") (net 1))
   (segment (start 148.76 112.272) (end 148.76 112.8346) (width 0.25) (layer "F.Cu") (net 1))
@@
   (segment (start 147.86 107.93) (end 148.61 107.93) (width 0.25) (layer "F.Cu") (net 1))
   (segment (start 144.0078 107.0179) (end 144.9199 107.93) (width 0.25) (layer "F.Cu") (net 1))
-  (segment (start 130.7947 115.4399) (end 130.887 115.4399) (width 0.25) (layer "F.Cu") (net 1))
   (segment (start 151.6788 102.2339) (end 151.48 102.0351) (width 0.25) (layer "F.Cu") (net 1))
   (segment (start 154.94 105.87) (end 156.0001 105.87) (width 0.25) (layer "F.Cu") (net 1))
@@
   (segment (start 151.1349 105.6362) (end 151.1349 105.93) (width 0.25) (layer "F.Cu") (net 1))
   (segment (start 165.1 105.8496) (end 156.0205 105.8496) (width 0.25) (layer "F.Cu") (net 1))
+  (segment (start 130.5162 111.665) (end 139.515 111.665) (width 0.25) (layer "F.Cu") (net 1))
   (segment (start 156.4275 116.84) (end 155.7149 116.84) (width 0.25) (layer "F.Cu") (net 1))
   (segment (start 154.8275 116.84) (end 155.7149 116.84) (width 0.25) (layer "F.Cu") (net 1))
@@
   (segment (start 150.61 105.93) (end 151.1349 105.93) (width 0.25) (layer "F.Cu") (net 1))
   (segment (start 149.86 106.68) (end 150.61 105.93) (width 0.25) (layer "F.Cu") (net 1))
+  (segment (start 130.887 115.4399) (end 130.7947 115.4399) (width 0.25) (layer "F.Cu") (net 1))
   (segment (start 130.887 116.915) (end 130.887 116.1774) (width 0.25) (layer "F.Cu") (net 1))
   (segment (start 145.4172 116.1774) (end 146.6317 114.9629) (width 0.25) (layer "F.Cu") (net 1))
   (segment (start 151.48 100.975) (end 151.48 102.0351) (width 0.25) (layer "F.Cu") (net 1))
   (segment (start 154.8275 116.84) (end 154.8275 117.1026) (width 0.25) (layer "F.Cu") (net 1))
-  (segment (start 130.887 116.1774) (end 130.887 115.4399) (width 0.25) (layer "F.Cu") (net 1))
+  (segment (start 129.4119 114.0571) (end 129.4119 112.7693) (width 0.25) (layer "F.Cu") (net 1))
   (segment (start 151.86 105.93) (end 151.1349 105.93) (width 0.25) (layer "F.Cu") (net 1))
   (segment (start 140.1691 104.2498) (end 138.9 102.9807) (width 0.25) (layer "F.Cu") (net 2))
@@
   (segment (start 148.4912 104.68) (end 147.86 105.3112) (width 0.25) (layer "F.Cu") (net 2))
   (segment (start 138.9 102.64) (end 138.9 102.9807) (width 0.25) (layer "F.Cu") (net 2))
+  (segment (start 142.494 100.584) (end 133.218 100.584) (width 0.25) (layer "F.Cu") (net 3))
   (segment (start 149.61 103.9549) (end 148.2951 102.64) (width 0.25) (layer "F.Cu") (net 3))
-  (segment (start 132.0621 101.7399) (end 143.53 101.7399) (width 0.25) (layer "F.Cu") (net 3))
+  (segment (start 143.53 102.64) (end 143.53 101.62) (width 0.25) (layer "F.Cu") (net 3))
   (segment (start 148.2951 102.64) (end 143.53 102.64) (width 0.25) (layer "F.Cu") (net 3))
-  (segment (start 130.887 102.915) (end 132.0621 101.7399) (width 0.25) (layer "F.Cu") (net 3))
-  (segment (start 143.53 102.64) (end 143.53 101.7399) (width 0.25) (layer "F.Cu") (net 3))
+  (segment (start 133.218 100.584) (end 130.887 102.915) (width 0.25) (layer "F.Cu") (net 3))
+  (segment (start 143.53 101.62) (end 142.494 100.584) (width 0.25) (layer "F.Cu") (net 3))
   (segment (start 149.61 104.68) (end 149.61 103.9549) (width 0.25) (layer "F.Cu") (net 3))
   (segment (start 148.502 102.1751) (end 150.11 103.7831) (width 0.25) (layer "F.Cu") (net 4))
